Commit message: Updated program for real time inference

File: src/vision_pipeline/urdf/hexacopter.urdf (robot description, URDF)
Before this commit: robot vtol_vision_rig, 2 links, 1 joints
Joints:
- joint camera_mount_joint: origin xyz=0.15 0.0 -0.05 rpy=0.0 0.349 0.0 -> xyz=-0.127 0.0 -0.1524 rpy=0.0 1.5708 0.0
